File: Hardware/CAN/EGT.kicad_pcb (KiCad board)
At the start: 2 copper layers, 18.6 x 14.6 mm, 22 parts, among them P1 CONN_4, P2 CONN_2, U1 MC33269, U2 PIC12F1840, U3 TJA1051TK/3, U4 AD8628

Commit message: Final routing
Parts:
- moved R6 15.1 mm to (149.9, 147.3), turned to 180 degrees
- moved R7 11.7 mm to (152.9, 147.3), turned to 90 degrees
- moved C8 11.2 mm to (154.8, 147.3), turned to 90 degrees
- moved U3 7.60 mm to (160.5, 156.6)
Routing:
- net N-000008: track 14.3 -> 92.6 mm, vias 2 -> 4
- net N-000006: track 19.8 -> 76.2 mm, vias 1 -> 4
- net N-0000013: track 0.00 -> 20.3 mm
- net N-0000010: track 0.00 -> 14.4 mm
- net N-000001: track 0.00 -> 12.4 mm, vias 0 -> 1
- net N-000003: track 0.00 -> 12.3 mm, vias 0 -> 1
- net N-000005: track 0.00 -> 9.77 mm, vias 0 -> 1
- net N-0000015: track 0.00 -> 9.67 mm
- net N-0000016: track 0.00 -> 7.83 mm
- net N-000009: track 0.00 -> 6.88 mm
- net N-000002: track 0.00 -> 4.48 mm
- net N-0000017: track 0.00 -> 2.06 mm
- net N-0000014: track 0.00 -> 2.06 mm
Other:
- net class Default: clearance 0.254 -> 0.155; trace_width 0.254 -> 0.2; via_dia 0.889 -> 0.7; via_drill 0.635 -> 0.6
- rule trace_clearance: 0.254 -> 0.155
